Commit message: Update farming_robot.xacro

File: farming_robot.xacro (robot description, xacro)
@@ -19,11 +19,11 @@
         <inertial>
             <origin xyz="0 0 0.5" rpy="0 0 0"/>
-            <mass value="1"/>
-            <inertia ixx="100"  ixy="0"  ixz="0" iyy="100" iyz="0" izz="100" />
+            <mass value="20"/>
+            <inertia ixx="0"  ixy="0"  ixz="0" iyy="1.6" iyz="1.6" izz="1" />
         </inertial>
         <visual>
             <origin rpy="0 0 0" xyz="0 0 0.4"/>
             <geometry>
-                <cylinder radius="0.40" length="0.8"/>
+                <cylinder radius="0.4" length="0.8"/>
             </geometry>
         </visual>
@@ -31,5 +31,5 @@
             <origin xyz="0 0 0" rpy="0 0 0"/>
             <geometry>
-                <cylinder radius="1" length="0.5"/>
+                <cylinder radius="0.4" length="0.8"/>
             </geometry>
         </collision>
@@ -45,6 +45,6 @@
         <inertial>
             <origin xyz="0 0 0.5" rpy="0 0 0"/>
-            <mass value="1"/>
-            <inertia ixx="100"  ixy="0"  ixz="0" iyy="100" iyz="0" izz="100" />
+            <mass value="10"/>
+            <inertia ixx="0"  ixy="0"  ixz="0" iyy="0.1125" iyz="0.1125" izz="1" />
         </inertial>
         <visual>
@@ -57,5 +57,5 @@
             <origin xyz="0 0 0" rpy="0 0 0"/>
             <geometry>
-                <cylinder radius="1" length="0.5"/>
+                <cylinder radius="0.15" length="0.8"/>
             </geometry>
         </collision>
@@ -71,6 +71,6 @@
         <inertial>
             <origin xyz="0 0 0.5" rpy="0 0 0"/>
-            <mass value="1"/>
-            <inertia ixx="100"  ixy="0"  ixz="0" iyy="100" iyz="0" izz="100" />
+            <mass value="10"/>
+            <inertia ixx="0"  ixy="0"  ixz="0" iyy="0.05" iyz="0.05" izz="1" />
         </inertial>
         <visual>
@@ -83,5 +83,5 @@
             <origin xyz="0 0 0" rpy="0 0 0"/>
             <geometry>
-                <cylinder radius="1" length="0.5"/>
+                <cylinder radius="0.1" length="0.7"/>
             </geometry>
         </collision>
@@ -97,6 +97,6 @@
         <inertial>
             <origin xyz="0 0 0.5" rpy="0 0 0"/>
-            <mass value="1"/>
-            <inertia ixx="100"  ixy="0"  ixz="0" iyy="100" iyz="0" izz="100" />
+            <mass value="10"/>
+            <inertia ixx="0"  ixy="0"  ixz="0" iyy="0.018" iyz="0.018" izz="1" />
         </inertial>
         <visual>
@@ -109,5 +109,5 @@
             <origin xyz="0 0 0" rpy="0 0 0"/>
             <geometry>
-                <cylinder radius="1" length="0.5"/>
+                <cylinder radius="0.06" length="0.6"/>
             </geometry>
         </collision>
@@ -123,6 +123,6 @@
         <inertial>
             <origin xyz="0 0 0.5" rpy="0 0 0"/>
-            <mass value="1"/>
-            <inertia ixx="100"  ixy="0"  ixz="0" iyy="100" iyz="0" izz="100" />
+            <mass value="10"/>
+            <inertia ixx="0"  ixy="0"  ixz="0" iyy="0.1125" iyz="0.1125" izz="100" />
         </inertial>
         <visual>
@@ -135,5 +135,5 @@
             <origin xyz="0 0 0" rpy="0 0 0"/>
             <geometry>
-                <cylinder radius="1" length="0.5"/>
+                <cylinder radius="0.15" length="0.8"/>
             </geometry>
         </collision>
@@ -149,6 +149,6 @@
         <inertial>
             <origin xyz="0 0 0.5" rpy="0 0 0"/>
-            <mass value="1"/>
-            <inertia ixx="100"  ixy="0"  ixz="0" iyy="100" iyz="0" izz="100" />
+            <mass value="10"/>
+            <inertia ixx="0"  ixy="0"  ixz="0" iyy="0.05" iyz="0" izz="10" />
         </inertial>
         <visual>
@@ -161,5 +161,5 @@
             <origin xyz="0 0 0" rpy="0 0 0"/>
             <geometry>
-                <cylinder radius="1" length="0.5"/>
+                <cylinder radius="0.10" length="0.7"/>
             </geometry>
         </collision>
@@ -175,6 +175,6 @@
         <inertial>
             <origin xyz="0 0 0.5" rpy="0 0 0"/>
-            <mass value="1"/>
-            <inertia ixx="100"  ixy="0"  ixz="0" iyy="100" iyz="0" izz="100" />
+            <mass value="10"/>
+            <inertia ixx="0"  ixy="0"  ixz="0" iyy="0.018" iyz="0.018" izz="1" />
         </inertial>
         <visual>
@@ -187,5 +187,5 @@
             <origin xyz="0 0 0" rpy="0 0 0"/>
             <geometry>
-                <cylinder radius="1" length="0.5"/>
+                <cylinder radius="0.06" length="0.6"/>
             </geometry>
         </collision>
